Commit message: 将 URDF 改为 xacro，支持 use_sim 条件编译，用于仿真/实车切换
给所有 world 文件添加 gazebo_ros_factory 插件，修复 /spawn_entity 服务不可用

重构启动文件：统一 use_sim_time 参数，使用 OpaqueFunction 确保参数正确解析，增加 standalone 参数避免 map->odom 双发布

添加 AGENTS.md，记录项目架构、启动命令和常见问题

参照模板编写 README 和项目详细文档

更新 AGENTS.md，引用 docs/details.md

添加 fix 分支修改记录，描述相对 main 的全部改动

统一文档路径为原仓库名 ros2_car，完善环境要求和文档引用

File: src/ros_car/urdf/ros_car.urdf.xacro (robot description, xacro)
@@ -1,4 +1,5 @@
 <?xml version="1.0" ?>
-<robot name="ros_car">
+<robot xmlns:xacro="http://www.ros.org/wiki/xacro" name="ros_car">
+  <xacro:property name="use_sim" value="true"/>
   <!-- ======== Materials ======== -->
   <material name="blue">  <color rgba="0.2 0.5 0.8 1.0"/></material>
@@ -26,7 +27,9 @@
     </inertial>
   </link>
+  <xacro:if value="${use_sim}">
   <gazebo reference="base_link">
     <mu1>0.5</mu1><mu2>0.5</mu2>
   </gazebo>
+  </xacro:if>
   <!-- ============================================================ -->
   <!--  LASER SENSOR                                                -->
@@ -72,4 +75,5 @@
     <origin rpy="0 0 0" xyz="0 0 0.04"/>
   </joint>
+  <xacro:if value="${use_sim}">
   <gazebo reference="laser_link">
     <sensor name="laser" type="ray">
@@ -104,4 +108,5 @@
     </sensor>
   </gazebo>
+  </xacro:if>
   <!-- ============================================================ -->
   <!--  IMU SENSOR                                                  -->
@@ -127,4 +132,5 @@
     <origin rpy="0 0 0" xyz="0 0 0.02"/>
   </joint>
+  <xacro:if value="${use_sim}">
   <gazebo reference="imu_link">
     <sensor name="imu_sensor" type="imu">
@@ -138,4 +144,5 @@
     </sensor>
   </gazebo>
+  </xacro:if>
   <!-- ============================================================ -->
   <!--  DUMMY STEERING WHEEL (cosmetic)                             -->
@@ -293,4 +300,5 @@
   </joint>
   <!-- Wheel friction for Gazebo -->
+  <xacro:if value="${use_sim}">
   <gazebo reference="left_front_link">
     <mu1>1.0</mu1><mu2>1.0</mu2>
@@ -309,7 +317,9 @@
     <material>Gazebo/Black</material>
   </gazebo>
+  </xacro:if>
   <!-- ============================================================ -->
   <!--  ACKERMANN DRIVE CONTROLLER                                  -->
   <!-- ============================================================ -->
+  <xacro:if value="${use_sim}">
   <gazebo>
     <plugin filename="libgazebo_ros_ackermann_drive.so" name="ackermann_controller">
@@ -340,3 +350,4 @@
     </plugin>
   </gazebo>
+  </xacro:if>
 </robot>
